File: _02-realisation/_02-hardware/usb5v3a_v2/usb5v3a_v2.kicad_sch (KiCad schematic)
At the start: 11 parts, among them J1 Conn_01x02_Male, J2 Conn_01x02_Male, U1 LM7805_TO220, U2 LM741, U3 INA219Module, U4 INA219Module, U5 OLED128x32

Commit message: USB 2x 3A v2 presque fini
Other:
- company: (none) -> VOROBOTICS
- title: (none) -> USB5V 3A 2 voies avec affichage du courant
Changed lines of the file:
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@@
 (kicad_sch (version 20211123) (generator eeschema)
   (paper "A4")
+  (title_block
+    (title "USB5V 3A 2 voies avec affichage du courant")
+    (date "07/10/2022")
+    (rev "1")
+    (company "VOROBOTICS")
+  )
   (junction (at 118.11 139.7) (diameter 0) (color 0 0 0 0)
   )
